Commit message: URDF w Gazebo and LM Design

File: description/robot_core.xacro (robot description, xacro)
@@ -4,5 +4,5 @@
     <xacro:include filename="inertial_macros.xacro"/>
     <material name="white">
-        <color rgba="1 1 1 1"/>
+        <color rgba="1 1 1 0.3"/>
     </material>
     <material name="orange">
@@ -10,9 +10,12 @@
     </material>
     <material name="blue">
-        <color rgba="0.2 0.2 1 1"/>
+        <color rgba="0.2 0.2 1 0.9"/>
     </material>
     <material name="black">
         <color rgba="0 0 0 1"/>
     </material>
+    <material name="grey">
+        <color rgba="0.2 0 0 1"/>
+    </material>
     <!-- Base Link -->
     <link name="base_link">
@@ -22,75 +25,204 @@
         <parent link="base_link"/>
         <child link="chassis"/>
-        <origin xyz="-0.1 0 0"/>
+        <origin xyz="-1.5 0 0"/>
     </joint>
     <link name="chassis">
         <visual>
-            <origin xyz="0.15 0 0.075"/>
-            <geometry>
-                <box size="0.3 0.3 0.15"/>
+            <origin xyz="1.5 0 0.5"/>
+            <geometry>
+                <box size="3 2 1"/>
             </geometry>
             <material name="white"/>
         </visual>
         <collision>
-            <origin xyz="0.15 0 0.075"/>
-            <geometry>
-                <box size="0.3 0.3 0.15"/>
+            <origin xyz="1.5 0 0.5"/>
+            <geometry>
+                <box size="3 2 1"/>
             </geometry>
             <material name="white"/>
         </collision>
-        <xacro:inertial_box mass="0.5" x="0.3" y="0.3" z="0.15">
-            <origin xyz="0.15 0 0.075" rpy="0 0 0"/>
+        <xacro:inertial_box mass="0.5" x="3" y="2" z="1">
+            <origin xyz="1.5 0 0.5" rpy="0 0 0"/>
         </xacro:inertial_box>
     </link>
-    <!-- Left Wheel -->
-    <joint name="left_wheel_joint" type="continuous">
-        <parent link="base_link"/>
-        <child link="left_wheel"/>
-        <origin xyz="0 0.175 0" rpy="-${pi/2} 0 0"/>
+    <!-- Left Wheel Rear -->
+    <joint name="left_wheel_rear_joint" type="continuous">
+        <parent link="base_link"/>
+        <child link="left_wheel_rear"/>
+        <origin xyz="-1 0.75 0" rpy="-${pi/2} 0 0"/>
         <axis xyz="0 0 1"/>
     </joint>
-    <link name="left_wheel">
-        <visual>
-            <geometry>
-                <cylinder length="0.04" radius="0.05" />/>
-            </geometry>
-            <material name="blue"/>
-        </visual>
-        <collision>
-            <geometry>
-                <cylinder length="0.04" radius="0.05" />/>
-            </geometry>
-            <material name="blue"/>
-        </collision>
-        <xacro:inertial_cylinder mass="0.1" length="0.05" radius="0.05">
+    <link name="left_wheel_rear">
+        <visual>
+            <geometry>
+                <cylinder length="0.2" radius="0.4" />/>
+            </geometry>
+            <material name="blue"/>
+        </visual>
+        <collision>
+            <geometry>
+                <cylinder length="0.2" radius="0.4" />/>
+            </geometry>
+            <material name="blue"/>
+        </collision>
+        <xacro:inertial_cylinder mass="0.1" length="0.2" radius="0.4">
             <origin xyz="0 0 0" rpy="0 0 0"/>
         </xacro:inertial_cylinder>
     </link>
     <!-- Right Wheel -->
-    <joint name="right_wheel_joint" type="continuous">
-        <parent link="base_link"/>
-        <child link="right_wheel"/>
-        <origin xyz="0 -0.175 0" rpy="${pi/2} 0 0"/>
-        <axis xyz="0 0 -1"/>
-    </joint>
-    <link name="right_wheel">
-        <visual>
-            <geometry>
-                <cylinder length="0.04" radius="0.05" />/>
-            </geometry>
-            <material name="blue"/>
-        </visual>
-        <collision>
-            <geometry>
-                <cylinder length="0.04" radius="0.05" />/>
-            </geometry>
-            <material name="blue"/>
-        </collision>
-        <xacro:inertial_sphere mass="0.1" radius="0.05">
-            <origin xyz="0 0 0" rpy="0 0 0"/>
-        </xacro:inertial_sphere>
-    </link>
-    <!-- Caster Wheel -->
-    <joint name="caster_wheel_joint" type="fixed">
+    <joint name="right_wheel_rear_joint" type="continuous">
+        <parent link="base_link"/>
+        <child link="right_wheel_rear"/>
+        <origin xyz="-1 -0.75 0" rpy="${pi/2} 0 0"/>
+        <axis xyz="0 0 -1"/>
+    </joint>
+    <link name="right_wheel_rear">
+        <visual>
+            <geometry>
+                <cylinder length="0.2" radius="0.4" />/>
+            </geometry>
+            <material name="blue"/>
+        </visual>
+        <collision>
+            <geometry>
+                <cylinder length="0.2" radius="0.4" />/>
+            </geometry>
+            <material name="blue"/>
+        </collision>
+        <xacro:inertial_cylinder mass="0.1" length="0.2" radius="0.4">
+            <origin xyz="0 0 0" rpy="0 0 0"/>
+        </xacro:inertial_cylinder>
+    </link>
+    <joint name="right_wheel_front_steer_joint" type="continuous">
+        <parent link="base_link"/>
+        <child link="right_wheel_front_steer"/>
+        <origin xyz="1 -0.75 0.5"/>
+        <axis xyz="0 0 -1"/>
+    </joint>
+    <link name="right_wheel_front_steer">
+        <visual>
+            <geometry>
+                <cylinder length="0.2" radius="0.02" />/>
+            </geometry>
+            <material name="grey"/>
+        </visual>
+        <collision>
+            <geometry>
+                <cylinder length="0.2" radius="0.02" />/>
+            </geometry>
+            <material name="grey"/>
+        </collision>
+        <xacro:inertial_cylinder mass="0.00001" length="0.2" radius="0.02">
+            <origin xyz="0 0 0" rpy="0 0 0"/>
+        </xacro:inertial_cylinder>
+    </link>
+    <joint name="right_wheel_front_joint" type="continuous">
+        <parent link="right_wheel_front_steer"/>
+        <child link="right_wheel_front"/>
+        <origin xyz="0 0 -0.5" rpy="${pi/2} 0 0"/>
+        <axis xyz="0 0 -1"/>
+    </joint>
+    <link name="right_wheel_front">
+        <visual>
+            <geometry>
+                <cylinder length="0.2" radius="0.4" />/>
+            </geometry>
+            <material name="blue"/>
+        </visual>
+        <collision>
+            <geometry>
+                <cylinder length="0.2" radius="0.4" />/>
+            </geometry>
+            <material name="blue"/>
+        </collision>
+        <xacro:inertial_cylinder mass="0.1" length="0.2" radius="0.4">
+            <origin xyz="0 0 0" rpy="0 0 0"/>
+        </xacro:inertial_cylinder>
+    </link>
+ <joint name="left_wheel_front_steer_joint" type="continuous">
+        <parent link="base_link"/>
+        <child link="left_wheel_front_steer"/>
+        <origin xyz="1 0.75 0.5"/>
+        <axis xyz="0 0 -1"/>
+    </joint>
+    <link name="left_wheel_front_steer">
+        <visual>
+            <geometry>
+                <cylinder length="0.2" radius="0.02" />/>
+            </geometry>
+            <material name="grey"/>
+        </visual>
+        <collision>
+            <geometry>
+                <cylinder length="0.2" radius="0.02" />/>
+            </geometry>
+            <material name="grey"/>
+        </collision>
+        <xacro:inertial_cylinder mass="0.0001" length="0.2" radius="0.02">
+            <origin xyz="0 0 0" rpy="0 0 0"/>
+        </xacro:inertial_cylinder>
+    </link>
+    <joint name="caster_wheel_joint" type="continuous">
+        <parent link="left_wheel_front_steer"/>
+        <child link="caster_wheel"/>
+        <origin xyz="0 0 -0.5" rpy="${pi/2} 0 0"/>
+        <axis xyz="0 0 -1"/>
+    </joint>
+    <link name="caster_wheel">
+        <visual>
+            <geometry>
+                <cylinder length="0.2" radius="0.4" />/>
+            </geometry>
+            <material name="blue"/>
+        </visual>
+        <collision>
+            <geometry>
+                <cylinder length="0.2" radius="0.4" />/>
+            </geometry>
+            <material name="blue"/>
+        </collision>
+        <xacro:inertial_cylinder mass="0.1" length="0.2" radius="0.4">
+            <origin xyz="0 0 0" rpy="0 0 0"/>
+        </xacro:inertial_cylinder>
+    </link>
+    <!--
+    <joint name="left_steering_joint">
+        <parent link="base_link"/>
+        <child link="left_steering"/>
+        <origin xyz="-1 -0.75 0"/>
+        <axis xyz="0 0 0"/>
+    </joint>
+    <link name="left_steering">
+        <visual>
+            <geometry>
+                <box size="0.3 0.2 0.1"/>
+            </geometry>
+            <material name="white"/>
+        </visual>
+    </link>
+    <joint name="left_wheel_front_joint" type="continuous">
+        <parent link="base_link"/>
+        <child link="left_wheel_rear"/>
+        <origin xyz="-1 0.75 0" rpy="-${pi/2} 0 0"/>
+        <axis xyz="0 0 1"/>
+    </joint>
+    <link name="left_wheel_rear">
+        <visual>
+            <geometry>
+                <cylinder length="0.2" radius="0.4" />/>
+            </geometry>
+            <material name="blue"/>
+        </visual>
+        <collision>
+            <geometry>
+                <cylinder length="0.2" radius="0.4" />/>
+            </geometry>
+            <material name="blue"/>
+        </collision>
+        <xacro:inertial_cylinder mass="0.1" length="0.2" radius="0.4">
+            <origin xyz="0 0 0" rpy="0 0 0"/>
+        </xacro:inertial_cylinder>
+    </link>
+        <joint name="caster_wheel_joint" type="fixed">
         <parent link="chassis"/>
         <child link="caster_wheel"/>
@@ -111,3 +243,4 @@
         </collision>
     </link>
+-->
 </robot>
