Commit message: gazibo auto launch

File: description/robot.urdf.xacro (robot description, xacro)
@@ -3,3 +3,4 @@
     <!-- Run other File -->
     <xacro:include filename="robot_core.xacro"/>
+    <xacro:include filename="gazebo_control.xacro"/>
 </robot>

File: description/robot_core.xacro (robot description, xacro)
@@ -25,5 +25,5 @@
         <parent link="base_link"/>
         <child link="chassis"/>
-        <origin xyz="-1.5 0 0"/>
+        <origin xyz="-1.5 0 0.5"/>
     </joint>
     <link name="chassis">
@@ -31,5 +31,5 @@
             <origin xyz="1.5 0 0.5"/>
             <geometry>
-                <box size="3 2 1"/>
+                <box size="3 1.25 1"/>
             </geometry>
             <material name="white"/>
@@ -50,5 +50,5 @@
         <parent link="base_link"/>
         <child link="left_wheel_rear"/>
-        <origin xyz="-1 0.75 0" rpy="-${pi/2} 0 0"/>
+        <origin xyz="-1 0.75 0.5" rpy="-${pi/2} 0 0"/>
         <axis xyz="0 0 1"/>
     </joint>
@@ -74,5 +74,5 @@
         <parent link="base_link"/>
         <child link="right_wheel_rear"/>
-        <origin xyz="-1 -0.75 0" rpy="${pi/2} 0 0"/>
+        <origin xyz="-1 -0.75 0.5" rpy="${pi/2} 0 0"/>
         <axis xyz="0 0 -1"/>
     </joint>
@@ -97,5 +97,5 @@
         <parent link="base_link"/>
         <child link="right_wheel_front_steer"/>
-        <origin xyz="1 -0.75 0.5"/>
+        <origin xyz="1 -0.75 1"/>
         <axis xyz="0 0 -1"/>
     </joint>
@@ -143,5 +143,5 @@
         <parent link="base_link"/>
         <child link="left_wheel_front_steer"/>
-        <origin xyz="1 0.75 0.5"/>
+        <origin xyz="1 0.75 1"/>
         <axis xyz="0 0 -1"/>
     </joint>
