Commit message: akermin drive

File: description/gazebo_control.xacro (robot description, xacro)
@@ -1,11 +1,30 @@
 <?xml version="1.0"?>
 <robot xmlns:xacro="http://www.ros.org/wiki/xacro"  name="robot">
+    <xacro:property name="wheel_friction" value="1"/>
+    <gazebo reference="front_left_wheel">
+        <mu1>${wheel_friction}</mu1>
+        <mu2>${wheel_friction}</mu2>
+        <material>Gazebo/DarkGrey</material>
+    </gazebo>
+    <gazebo reference="front_right_wheel">
+        <mu1>${wheel_friction}</mu1>
+        <mu2>${wheel_friction}</mu2>
+        <material>Gazebo/DarkGrey</material>
+    </gazebo>
+    <gazebo reference="back_left_wheel">
+        <mu1>${wheel_friction}</mu1>
+        <mu2>${wheel_friction}</mu2>
+        <material>Gazebo/DarkGrey</material>
+    </gazebo>
+    <gazebo reference="back_right_wheel">
+        <mu1>${wheel_friction}</mu1>
+        <mu2>${wheel_friction}</mu2>
+        <material>Gazebo/DarkGrey</material>
+    </gazebo>
+    <gazebo reference="odom">
+        <dampingFactor>0.00007</dampingFactor>
+    </gazebo>
     <gazebo>
-        <plugin name="diff_drgazebogazebo_ros_control" filename="libgazebo_ros_control.so">
-            <!-- Wheel Information -->
-            <robotNamesapce>/</robotNamesapce>
-            <robotSimType>steer_bot_hardware_gazebo/SteerBotHardwareGazebo</robotSimType>
-            <left_wheel_rear_joint>left_wheel_rear_joint</left_wheel_rear_joint>
-            <right_wheel_rear_joint>right_wheel_rear_joint</right_wheel_rear_joint>
+        <plugin name="car_gazebo_plugin" filename="libcar_gazebo_plugin.so">
         </plugin>
     </gazebo>

File: description/robot.urdf.xacro (robot description, xacro)
@@ -4,3 +4,6 @@
     <xacro:include filename="robot_core.xacro"/>
     <xacro:include filename="gazebo_control.xacro"/>
+            <!--
+    <xacro:include filename="lidar.xacro"/>
+    -->
 </robot>

File: description/robot_core.xacro (robot description, xacro)
@@ -1,246 +1,353 @@
 <?xml version="1.0"?>
-<robot xmlns:xacro="http://www.ros.org/wiki/xacro" >
-    <!-- Include Inertial File -->
-    <xacro:include filename="inertial_macros.xacro"/>
-    <material name="white">
-        <color rgba="1 1 1 0.3"/>
+<robot xmlns:xacro="http://www.ros.org/wiki/xacro"  name="robot">
+  <xacro:arg name="wheel_diameter" default="0.254"/>
+  <xacro:property name="wheel_radius" value="${$(arg wheel_diameter)/2}"/>
+  <xacro:property name="wheel_width" value="0.05"/>
+  <xacro:property name="wheelbase_length" value="0.6096"/>
+  <xacro:property name="front_wheelbase_width" value="0.4572"/>
+  <xacro:property name="rear_wheelbase_width" value="0.4572"/>
+  <xacro:property name="wheel_mass" value="1"/>
+  <xacro:property name="total_mass" value = "5.0"/>
+  <xacro:property name="shock_travel" value = "0.035"/>
+  <xacro:property name="shock_height" value = "0.2"/>
+  <xacro:property name="chassis_height" value = "0.0254"/>
+  <xacro:property name="chassis_elevation" value = "0.3"/>
+  <xacro:property name="chassis_mass" value = "${total_mass-4*wheel_mass}"/>
+  <xacro:property name="chassis_l" value = "0.9144"/>
+  <xacro:property name="chassis_w" value = "0.6096"/>
+  <xacro:property name="chassis_t" value = "0.0254"/>
+  <xacro:property name="steering_limit" value = "1"/>
+  <xacro:macro name="cylinder_inertia" params="m r h">
+        <inertia  ixx="${m*(3*r*r+h*h)/12}" ixy = "0" ixz = "0"
+                    iyy="${m*(3*r*r+h*h)/12}" iyz = "0"
+                    izz="${m*r*r/2}" />
+  </xacro:macro>
+  <xacro:macro name="box_inertia" params="m x y z">
+          <inertia  ixx="${m*(y*y+z*z)/12}" ixy = "0" ixz = "0"
+                    iyy="${m*(x*x+z*z)/12}" iyz = "0"
+                    izz="${m*(x*x+z*z)/12}" />
+  </xacro:macro>
+  <xacro:macro name="sphere_inertia" params="m r">
+          <inertia  ixx="${2*m*r*r/5}" ixy = "0" ixz = "0"
+                    iyy="${2*m*r*r/5}" iyz = "0"
+                    izz="${2*m*r*r/5}" />
+  </xacro:macro>
+  <xacro:macro name="cylinder_inertial" params="m r h">
+    <inertial>
+      <mass value="${m}"/>
+      <xacro:cylinder_inertia m="${m}" r="${r}" h="${h}"/>
+    </inertial>
+  </xacro:macro>
+  <link name="base_footprint"/>
+  <link name="base_link"/>
+<!--
+  <link name="base_link">
+    <visual>
+      <origin xyz="0 0 0.1" rpy="0 0 0"/>
+      <geometry>
+        <cylinder length="0.2" radius="0.01"/>
+      </geometry>
+      <material name="silver">
+        <color rgba="0.75 0.75 0.75 1"/>
+      </material>
+    </visual>
+    <collision>
+      <origin xyz="0 0 0.1" rpy="0 0 0"/>
+      <geometry>
+        <cylinder length="0.2" radius="0.01"/>
+      </geometry>
+    </collision>
+    <inertial>
+      <mass value="0.01"/>
+      <inertia ixx="0.015" iyy="0.0375" izz="0.0375"
+               ixy="0" ixz="0" iyz="0"/>
+    </inertial>
+  </link>
+-->
+  <link name="chassis_link">
+    <visual>
+      <geometry>
+        <box size="${chassis_l} ${chassis_w} ${chassis_t}"/>
+      </geometry>
+    </visual>
+    <collision>
+      <geometry>
+        <box size="${chassis_l} ${chassis_w} ${chassis_t}"/>
+      </geometry>
+    </collision>
+    <inertial>
+      <mass value="${chassis_mass}"/>
+      <xacro:box_inertia m="${chassis_mass}" x="${chassis_l}" y="${chassis_w}" z="${chassis_t}"/>
+    </inertial>
+  </link>
+  <link name="back_left_wheel">
+    <visual>
+      <geometry>
+        <cylinder length="${wheel_width}" radius="${wheel_radius}"/>
+      </geometry>
+      <material name="black">
+        <color rgba="0 0 0 1"/>
+      </material>
+    </visual>
+    <collision>
+      <geometry>
+        <cylinder length="${wheel_width}" radius="${wheel_radius}"/>
+      </geometry>
+    </collision>
+    <xacro:cylinder_inertial m="${wheel_mass}" r="${wheel_radius}" h="${wheel_width}"/>
+  </link>
+  <link name="back_right_wheel">
+    <visual>
+      <geometry>
+        <cylinder length="${wheel_width}" radius="${wheel_radius}"/>
+      </geometry>
+      <material name="black">
+        <color rgba="0 0 0 1"/>
+      </material>
+    </visual>
+    <collision>
+      <geometry>
+        <cylinder length="${wheel_width}" radius="${wheel_radius}"/>
+      </geometry>
+    </collision>
+    <xacro:cylinder_inertial m="${wheel_mass}" r="${wheel_radius}" h="${wheel_width}"/>
+  </link>
+  <link name="front_left_wheel_steer">
+    <visual>
+      <geometry>
+        <cylinder length="0.01" radius="0.01"/>
+      </geometry>
+      <material name="black">
+        <color rgba="0 0 0 1"/>
+      </material>
+    </visual>
+    <collision>
+      <geometry>
+        <cylinder length="0.01" radius="0.01"/>
+      </geometry>
+    </collision>
+    <inertial>
+      <mass value="0.1"/>
+      <inertia ixx="5.1458e-5" iyy="5.1458e-5" izz="6.125e-5"
+               ixy="0" ixz="0" iyz="0"/>
+    </inertial>
+  </link>
+    <link name="front_left_wheel">
+    <visual>
+      <geometry>
+        <cylinder length="${wheel_width}" radius="${wheel_radius}"/>
+      </geometry>
+      <material name="black">
+        <color rgba="0 0 0 1"/>
+      </material>
+    </visual>
+    <collision>
+      <geometry>
+        <cylinder length="${wheel_width}" radius="${wheel_radius}"/>
+      </geometry>
+    </collision>
+    <xacro:cylinder_inertial m="${wheel_mass}" r="${wheel_radius}" h="${wheel_width}"/>
+  </link>
+  <link name="front_right_wheel_steer">
+    <visual>
+      <geometry>
+        <cylinder length="0.01" radius="0.01"/>
+      </geometry>
+      <material name="black">
+        <color rgba="0 0 0 1"/>
+      </material>
+    </visual>
+    <collision>
+      <geometry>
+        <cylinder length="0.01" radius="0.01"/>
+      </geometry>
+    </collision>
+    <inertial>
+      <mass value="0.1"/>
+      <inertia ixx="5.1458e-5" iyy="5.1458e-5" izz="6.125e-5"
+               ixy="0" ixz="0" iyz="0"/>
+    </inertial>
+  </link>
+  <link name="front_right_wheel">
+    <visual>
+      <geometry>
+        <cylinder length="${wheel_width}" radius="${wheel_radius}"/>
+      </geometry>
+      <material name="black">
+        <color rgba="0 0 0 1"/>
+      </material>
+    </visual>
+    <collision>
+      <geometry>
+        <cylinder length="${wheel_width}" radius="${wheel_radius}"/>
+      </geometry>
+    </collision>
+    <xacro:cylinder_inertial m="${wheel_mass}" r="${wheel_radius}" h="${wheel_width}"/>
+  </link>
+  <link name="back_left_wheel_shock">
+      <visual>
+      <origin xyz="0 0 ${shock_height}" rpy="0 0 0"/>
+      <geometry>
+        <cylinder length="0.05" radius="0.01"/>
+      </geometry>
+      <material name="silver">
+        <color rgba="0.75 0.75 0.75 1"/>
+      </material>
+    </visual>
+    <collision>
+      <origin xyz="0 0 ${shock_height}" rpy="0 0 0"/>
+      <geometry>
+        <cylinder length="0.05" radius="0.01"/>
+      </geometry>
+    </collision>
+    <inertial>
+      <mass value="0.01"/>
+      <inertia ixx="0.015" iyy="0.0375" izz="0.0375"
+               ixy="0" ixz="0" iyz="0"/>
+    </inertial>
+  </link>
+  <link name="back_right_wheel_shock">
+    <visual>
+    <origin xyz="0 0 ${shock_height}" rpy="0 0 0"/>
+    <geometry>
+      <cylinder length="0.05" radius="0.01"/>
+    </geometry>
+    <material name="silver">
+      <color rgba="0.75 0.75 0.75 1"/>
     </material>
-    <material name="orange">
-        <color rgba="1 0.3 0.1 1"/>
-    </material>
-    <material name="blue">
-        <color rgba="0.2 0.2 1 0.9"/>
-    </material>
-    <material name="black">
-        <color rgba="0 0 0 1"/>
-    </material>
-    <material name="grey">
-        <color rgba="0.2 0 0 1"/>
-    </material>
-    <!-- Base Link -->
-    <link name="base_link">
-    </link>
-    <!-- Chassis Link -->
-    <joint name="chasis_joint" type="fixed">
-        <parent link="base_link"/>
-        <child link="chassis"/>
-        <origin xyz="-1.5 0 0.5"/>
-    </joint>
-    <link name="chassis">
-        <visual>
-            <origin xyz="1.5 0 0.5"/>
-            <geometry>
-                <box size="3 1.25 1"/>
-            </geometry>
-            <material name="white"/>
-        </visual>
-        <collision>
-            <origin xyz="1.5 0 0.5"/>
-            <geometry>
-                <box size="3 2 1"/>
-            </geometry>
-            <material name="white"/>
-        </collision>
-        <xacro:inertial_box mass="0.5" x="3" y="2" z="1">
-            <origin xyz="1.5 0 0.5" rpy="0 0 0"/>
-        </xacro:inertial_box>
-    </link>
-    <!-- Left Wheel Rear -->
-    <joint name="left_wheel_rear_joint" type="continuous">
-        <parent link="base_link"/>
-        <child link="left_wheel_rear"/>
-        <origin xyz="-1 0.75 0.5" rpy="-${pi/2} 0 0"/>
-        <axis xyz="0 0 1"/>
-    </joint>
-    <link name="left_wheel_rear">
-        <visual>
-            <geometry>
-                <cylinder length="0.2" radius="0.4" />/>
-            </geometry>
-            <material name="blue"/>
-        </visual>
-        <collision>
-            <geometry>
-                <cylinder length="0.2" radius="0.4" />/>
-            </geometry>
-            <material name="blue"/>
-        </collision>
-        <xacro:inertial_cylinder mass="0.1" length="0.2" radius="0.4">
-            <origin xyz="0 0 0" rpy="0 0 0"/>
-        </xacro:inertial_cylinder>
-    </link>
-    <!-- Right Wheel -->
-    <joint name="right_wheel_rear_joint" type="continuous">
-        <parent link="base_link"/>
-        <child link="right_wheel_rear"/>
-        <origin xyz="-1 -0.75 0.5" rpy="${pi/2} 0 0"/>
-        <axis xyz="0 0 -1"/>
-    </joint>
-    <link name="right_wheel_rear">
-        <visual>
-            <geometry>
-                <cylinder length="0.2" radius="0.4" />/>
-            </geometry>
-            <material name="blue"/>
-        </visual>
-        <collision>
-            <geometry>
-                <cylinder length="0.2" radius="0.4" />/>
-            </geometry>
-            <material name="blue"/>
-        </collision>
-        <xacro:inertial_cylinder mass="0.1" length="0.2" radius="0.4">
-            <origin xyz="0 0 0" rpy="0 0 0"/>
-        </xacro:inertial_cylinder>
-    </link>
-    <joint name="right_wheel_front_steer_joint" type="continuous">
-        <parent link="base_link"/>
-        <child link="right_wheel_front_steer"/>
-        <origin xyz="1 -0.75 1"/>
-        <axis xyz="0 0 -1"/>
-    </joint>
-    <link name="right_wheel_front_steer">
-        <visual>
-            <geometry>
-                <cylinder length="0.2" radius="0.02" />/>
-            </geometry>
-            <material name="grey"/>
-        </visual>
-        <collision>
-            <geometry>
-                <cylinder length="0.2" radius="0.02" />/>
-            </geometry>
-            <material name="grey"/>
-        </collision>
-        <xacro:inertial_cylinder mass="0.00001" length="0.2" radius="0.02">
-            <origin xyz="0 0 0" rpy="0 0 0"/>
-        </xacro:inertial_cylinder>
-    </link>
-    <joint name="right_wheel_front_joint" type="continuous">
-        <parent link="right_wheel_front_steer"/>
-        <child link="right_wheel_front"/>
-        <origin xyz="0 0 -0.5" rpy="${pi/2} 0 0"/>
-        <axis xyz="0 0 -1"/>
-    </joint>
-    <link name="right_wheel_front">
-        <visual>
-            <geometry>
-                <cylinder length="0.2" radius="0.4" />/>
-            </geometry>
-            <material name="blue"/>
-        </visual>
-        <collision>
-            <geometry>
-                <cylinder length="0.2" radius="0.4" />/>
-            </geometry>
-            <material name="blue"/>
-        </collision>
-        <xacro:inertial_cylinder mass="0.1" length="0.2" radius="0.4">
-            <origin xyz="0 0 0" rpy="0 0 0"/>
-        </xacro:inertial_cylinder>
-    </link>
- <joint name="left_wheel_front_steer_joint" type="continuous">
-        <parent link="base_link"/>
-        <child link="left_wheel_front_steer"/>
-        <origin xyz="1 0.75 1"/>
-        <axis xyz="0 0 -1"/>
-    </joint>
-    <link name="left_wheel_front_steer">
-        <visual>
-            <geometry>
-                <cylinder length="0.2" radius="0.02" />/>
-            </geometry>
-            <material name="grey"/>
-        </visual>
-        <collision>
-            <geometry>
-                <cylinder length="0.2" radius="0.02" />/>
-            </geometry>
-            <material name="grey"/>
-        </collision>
-        <xacro:inertial_cylinder mass="0.0001" length="0.2" radius="0.02">
-            <origin xyz="0 0 0" rpy="0 0 0"/>
-        </xacro:inertial_cylinder>
-    </link>
-    <joint name="caster_wheel_joint" type="continuous">
-        <parent link="left_wheel_front_steer"/>
-        <child link="caster_wheel"/>
-        <origin xyz="0 0 -0.5" rpy="${pi/2} 0 0"/>
-        <axis xyz="0 0 -1"/>
-    </joint>
-    <link name="caster_wheel">
-        <visual>
-            <geometry>
-                <cylinder length="0.2" radius="0.4" />/>
-            </geometry>
-            <material name="blue"/>
-        </visual>
-        <collision>
-            <geometry>
-                <cylinder length="0.2" radius="0.4" />/>
-            </geometry>
-            <material name="blue"/>
-        </collision>
-        <xacro:inertial_cylinder mass="0.1" length="0.2" radius="0.4">
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